Commit message: Simplify Gilbreth env for MOOC.

File: gilbreth_support/urdf/gilbreth.xacro (robot description, xacro)
@@ -6,8 +6,8 @@
   <xacro:include filename="$(find gilbreth_support)/urdf/bin/bin.urdf.xacro"/>
   <xacro:bin_urdf prefix="bin_1_"/>
-  <xacro:bin_urdf prefix="bin_2_"/>
+  <!-- <xacro:bin_urdf prefix="bin_2_"/>
   <xacro:bin_urdf prefix="bin_3_"/>
   <xacro:bin_urdf prefix="bin_4_"/>
-  <xacro:bin_urdf prefix="bin_5_"/>
+  <xacro:bin_urdf prefix="bin_5_"/> -->
   <!-- depth camera -->
   <xacro:include filename="$(find gilbreth_support)/urdf/depth_camera/depth_camera.urdf.xacro"/>
@@ -40,26 +40,26 @@
   </joint>
   <!-- a bin in the frame bin2_frame -->
-  <joint name="bin_2_joint" type="fixed">
+  <!-- <joint name="bin_2_joint" type="fixed">
     <parent link="world" />
     <child link="bin_2_base_link" />
     <origin xyz="-0.3 -0.4 0.0" rpy="0 0 0" />
-  </joint>
+  </joint> -->
   <!-- a bin in the frame bin3_frame -->
-  <joint name="bin_3_joint" type="fixed">
+  <!-- <joint name="bin_3_joint" type="fixed">
     <parent link="world" />
     <child link="bin_3_base_link" />
     <origin xyz="-0.3 0.4 0.0" rpy="0 0 0" />
-  </joint>
+  </joint> -->
   <!-- a bin in the frame bin4_frame -->
-  <joint name="bin_4_joint" type="fixed">
+  <!-- <joint name="bin_4_joint" type="fixed">
     <parent link="world" />
     <child link="bin_4_base_link" />
     <origin xyz="-0.3 1.2 0.0" rpy="0 0 0" />
-  </joint>
+  </joint> -->
   <!-- a bin in the frame bin5_frame -->
-  <joint name="bin_5_joint" type="fixed">
+  <!-- <joint name="bin_5_joint" type="fixed">
     <parent link="world" />
     <child link="bin_5_base_link" />
     <origin xyz="-0.3 -2.0 0.0" rpy="0 0 0" />
-  </joint>
+  </joint> -->
 </robot>

Commit message: Minor modification of bin position.

File: gilbreth_support/urdf/gilbreth.xacro (robot description, xacro)
@@ -6,8 +6,4 @@
   <xacro:include filename="$(find gilbreth_support)/urdf/bin/bin.urdf.xacro"/>
   <xacro:bin_urdf prefix="bin_1_"/>
-  <!-- <xacro:bin_urdf prefix="bin_2_"/>
-  <xacro:bin_urdf prefix="bin_3_"/>
-  <xacro:bin_urdf prefix="bin_4_"/>
-  <xacro:bin_urdf prefix="bin_5_"/> -->
   <!-- depth camera -->
   <xacro:include filename="$(find gilbreth_support)/urdf/depth_camera/depth_camera.urdf.xacro"/>
@@ -37,5 +33,5 @@
     <parent link="world" />
     <child link="bin_1_base_link" />
-    <origin xyz="-0.3 -1.2 0.0" rpy="0 0 0" />
+    <origin xyz="-1.8 -2.5 0.0" rpy="0 0 0" />
   </joint>
   <!-- a bin in the frame bin2_frame -->
